File: AccuracyAnalysis/architecture-schematics/naive-current-desensitized-architecture.kicad_sch (KiCad schematic)
At the start: 10 parts, among them Q1 Q_NMOS_GDS, U1 Adjustable_LDO

Commit message: add resistor-containing architecture
Parts:
- added RDesen2: R_US, symbol Device:R_US
- renumbered A1 to A2, BT1 to BT2, D1 to D2, MESA1 to MESA2, MESV1 to MESV2, Q1 to Q2, RAdjCharge1 to RAdjCharge2, RAdjDisch1 to RAdjDisch2, U1 to U2
Connections:
- net at MESA2.2 (+): now also RDesen2.1; no longer D2.2 (K)
- new net: RAdjCharge2. (R2), RfixedDiv2.2, U2. (VOUT)
- new net: D2.2 (K), RDesen2.2
Changed lines of the file:
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@@
-    (stroke (width 0) (type default) (color 0 0 0 0))
-  )
-  (wire (pts (xy 198.12 92.71) (xy 157.48 92.71))
     (stroke (width 0) (type default) (color 0 0 0 0))
   )
@@
     (stroke (width 0) (type default) (color 0 0 0 0))
   )
+  (wire (pts (xy 180.34 92.71) (xy 198.12 92.71))
+    (stroke (width 0) (type default) (color 0 0 0 0))
+  )
   (wire (pts (xy 171.45 111.76) (xy 171.45 114.3))
+    (stroke (width 0) (type default) (color 0 0 0 0))
+  )
+  (wire (pts (xy 172.72 92.71) (xy 157.48 92.71))
     (stroke (width 0) (type default) (color 0 0 0 0))
   )
@@
   (symbol (lib_id "MCU_Module:Arduino_UNO_R3") (at 125.73 97.79 0) (unit 1)
     (in_bom yes) (on_board yes)
-    (property "Reference" "A1" (id 0) (at 134.0994 72.39 0)
+    (property "Reference" "A2" (id 0) (at 134.0994 72.39 0)
       (effects (font (size 1.27 1.27)) (justify left))
     )
@@
   (symbol (lib_id "Rapid-EPS_architecture-blocks:Adjustable_LDO") (at 168.91 67.31 0) (unit 1)
     (in_bom yes) (on_board yes) (fields_autoplaced)
-    (property "Reference" "U1" (id 0) (at 168.91 67.31 0))
+    (property "Reference" "U2" (id 0) (at 168.91 67.31 0))
     (property "Value" "Adjustable_LDO" (id 1) (at 168.91 69.85 0))
     (property "Footprint" "" (id 2) (at 168.91 67.31 0)
@@
     (pin "")
   )
+  (symbol (lib_id "Device:R_US") (at 176.53 92.71 90) (unit 1)
+    (in_bom yes) (on_board yes) (fields_autoplaced)
+    (property "Reference" "RDesen2" (id 0) (at 176.53 86.36 90)
+      (effects (font (size 1.27 1.27)) hide)
+    )
+    (property "Value" "R_US" (id 1) (at 176.53 88.9 90)
+      (effects (font (size 1.27 1.27)) hide)
+    )
+    (property "Footprint" "" (id 2) (at 176.784 91.694 90)
+      (effects (font (size 1.27 1.27)) hide)
+    )
+    (property "Datasheet" "~" (id 3) (at 176.53 92.71 0)
+      (effects (font (size 1.27 1.27)) hide)
+    )
+    (pin "1")
+    (pin "2")
+  )
   (symbol (lib_id "Simulation_SPICE:DIODE") (at 198.12 80.01 270) (unit 1)
     (in_bom yes) (on_board yes)
-    (property "Reference" "D1" (id 0) (at 200.66 78.7399 90)
+    (property "Reference" "D2" (id 0) (at 200.66 78.7399 90)
       (effects (font (size 1.27 1.27)) (justify left))
     )
@@
   (symbol (lib_id "Rapid-EPS_architecture-blocks:Ammeter_DIO") (at 157.48 97.79 0) (unit 1)
     (in_bom yes) (on_board yes) (fields_autoplaced)
-    (property "Reference" "MESA1" (id 0) (at 161.29 96.0754 0)
+    (property "Reference" "MESA2" (id 0) (at 161.29 96.0754 0)
       (effects (font (size 1.27 1.27)) (justify left) hide)
     )
@@
   (symbol (lib_id "Device:Q_NMOS_GDS") (at 166.37 101.6 270) (unit 1)
     (in_bom yes) (on_board yes) (fields_autoplaced)
-    (property "Reference" "Q1" (id 0) (at 166.37 109.22 90)
+    (property "Reference" "Q2" (id 0) (at 166.37 109.22 90)
       (effects (font (size 1.27 1.27)) hide)
     )
@@
   (symbol (lib_id "Device:Battery_Cell") (at 161.29 110.49 0) (unit 1)
     (in_bom yes) (on_board yes) (fields_autoplaced)
-    (property "Reference" "BT1" (id 0) (at 165.1 107.1879 0)
+    (property "Reference" "BT2" (id 0) (at 165.1 107.1879 0)
       (effects (font (size 1.27 1.27)) (justify left) hide)
     )
@@
   (symbol (lib_name "digipot_1") (lib_id "Rapid-EPS_architecture-blocks:digipot") (at 185.42 107.95 0) (mirror y) (unit 1)
     (in_bom yes) (on_board yes) (fields_autoplaced)
-    (property "Reference" "RAdjDisch1" (id 0) (at 179.07 102.87 0)
+    (property "Reference" "RAdjDisch2" (id 0) (at 179.07 102.87 0)
       (effects (font (size 1.27 1.27)) hide)
     )
@@
   (symbol (lib_name "digipot_2") (lib_id "Rapid-EPS_architecture-blocks:digipot") (at 193.04 82.55 0) (mirror y) (unit 1)
     (in_bom yes) (on_board yes) (fields_autoplaced)
-    (property "Reference" "RAdjCharge1" (id 0) (at 187.96 77.47 0)
+    (property "Reference" "RAdjCharge2" (id 0) (at 187.96 77.47 0)
       (effects (font (size 1.27 1.27)) hide)
     )
@@
   (symbol (lib_id "Rapid-EPS_architecture-blocks:Voltmeter_DIO") (at 153.67 109.22 0) (unit 1)
     (in_bom yes) (on_board yes) (fields_autoplaced)
-    (property "Reference" "MESV1" (id 0) (at 157.48 107.5054 0)
-      (effects (font (size 1.27 1.27)) (justify left) hide)
-    )
+    (property "Reference" "MESV2" (id 0) (at 157.48 107.5054 0)
+      (effects (font (size 1.27 1.27)) (justify left) hide)
+    )
