File: Schematics/tester-schematic/tester-schematic.kicad_sch (KiCad schematic)
At the start: 5 parts, among them U1 ISL95810UIU8Z, U2 LT3741EFE#PBF

Commit message: work on schematic
Parts:
- removed C1: 1uF, CAPC2012X127N, symbol 0805cap:S-0805
- removed C2: 100uF, CAPC2012X127N, symbol 0805cap:S-0805
- removed L1: 560nH, IND_IHLP-6767GZ_VIS, symbol 560nH_IND:IHLP6767GZERR56M01
- removed U1: ISL95810UIU8Z, MSOP8_3P05X3P05_INR, symbol digipot:ISL95810UIU8Z
- removed U2: LT3741EFE#PBF, SOP65P640X120-20N, symbol Buck2:LT3741EFE#PBF
- added A?: Arduino_UNO_R3, Module:Arduino_UNO_R3, symbol MCU_Module:Arduino_UNO_R3
- added D?: VS-EPU6006L-N3, TO247AD_IXY, symbol 2022-05-28_06-14-30:VS-EPU6006L-N3
- added Q?: TPH3R704PC,LQ, TPH3R7_TOS, symbol Battery Tester Symbols:TPH3R704PC,LQ
- added R?: R_US, symbol Device:R_US
- added R?: TKH45PR050JE-TR, RES_TKH45_OHM, symbol Battery Tester Symbols:TKH45PR050JE-TR
- added U?: MAX5215GUA+, 21-0036K_MXM, symbol Battery Tester Symbols:MAX5215GUA+
- added U?: OPA2990IDR, D8_TEX, symbol Battery Tester Symbols:OPA2990IDR
- added U?: ISL95810UIU8Z, MSOP8_3P05X3P05_INR, symbol Battery Tester Symbols:ISL95810UIU8Z
- added U?: LT3741EFE-1-PBF, TSSOP20_FE_ADI, symbol Battery Tester Symbols:LT3741EFE-1-PBF
Connections:
- net Bench HV GND: now also A?.29 (GND), A?.6 (GND), A?.7 (GND), U?.2 (GND), U?.4 (GND), U?.5 (RW)
- net Bench HV PWR: now also D?.2
- net Bench LV PWR: now also A?.8 (VIN)
- new net: D?.1, U?.3 (VIN), U?.8 (V+)
- new net: A?.14 (SCL/A5), A?.32 (SCL/A5), U?.2 (SCL), U?.3 (SCL)
- new net: A?.13 (SDA/A4), A?.31 (SDA/A4), U?.3 (SDA), U?.4 (SDA)
- new net: A?.5 (+5V), U?.1 (*WP), U?.8 (VCC)
- new net: Q?.1, Q?.2, Q?.3
- new net: Q?.5, Q?.6, Q?.7, Q?.8, R?.1
- new net: R?.1, U?.18 (SW)
- new net: R?.2, U?.10 (FB), U?.6 (RL)
- no-connect marks 0 -> 1
